Commit message: Version 2.0: Complete working system with 6 demonstration videos
🎉 MAJOR UPDATE - WORKING VERSION 🎉

Robot Changes:
- Fixed 4-wheel design (2 driven front, 2 passive rear)
- Stable geometry, sits flat without tilting
- Proper differential drive turning
- All 4 wheels identical size (0.1m radius)

Path Execution:
- 9-cycle drive-stop-turn-stop pattern
- 100% success rate
- Complete CSV data logging
- Clear 1-second pauses between actions

New Files:
- simulation_run_4_working.mp4: 4-wheel robot demo
- simulation_run_5_working.mp4: 9-cycle execution
- simulation_run_6_final.mp4: Final validation
- follow_path_final.py: Working 9-cycle script
- CHANGELOG.md: Complete version history
- 3 new CSV data files from successful runs

Updated Files:
- ugress.urdf: Working 4-wheel configuration
- spawn_robot.launch: Clean working launch file
- videos/README.md: Updated with all 6 videos

Performance:
- Forward: 0.3 m/s stable
- Turning: 0.5 rad/s smooth 90° turns
- Success: 9/9 cycles completed (100%)

Status: ✅ THESIS READY
Tested: December 7-8, 2024
Result: 100% Success Rate

All code, videos, and documentation validated for thesis submission.

File: ugress_sim/urdf/ugress.urdf (robot description, URDF)
Before this commit: robot ugress, 4 links, 3 joints
Links:
- removed link caster_wheel
- removed link left_wheel
- removed link right_wheel
- added link front_left_wheel, mass 0.5; collision cylinder length=0.05 radius=0.1; visual cylinder length=0.05 radius=0.1
- added link front_right_wheel, mass 0.5; collision cylinder length=0.05 radius=0.1; visual cylinder length=0.05 radius=0.1
- added link rear_left_wheel, mass 0.5; collision cylinder length=0.05 radius=0.1; visual cylinder length=0.05 radius=0.1
- added link rear_right_wheel, mass 0.5; collision cylinder length=0.05 radius=0.1; visual cylinder length=0.05 radius=0.1
- link base_link: geometry collision box size=0.8 0.5 0.2; visual box size=0.8 0.5 0.2
Joints:
- removed joint caster_wheel_joint
- removed joint left_wheel_joint
- removed joint right_wheel_joint
- added joint front_left_wheel_joint: type continuous, parent base_link, child front_left_wheel, origin xyz=0.25 0.28 0 rpy=0 0 0, axis 0 1 0
- added joint front_right_wheel_joint: type continuous, parent base_link, child front_right_wheel, origin xyz=0.25 -0.28 0 rpy=0 0 0, axis 0 1 0
- added joint rear_left_wheel_joint: type continuous, parent base_link, child rear_left_wheel, origin xyz=-0.25 0.28 0 rpy=0 0 0, axis 0 1 0
- added joint rear_right_wheel_joint: type continuous, parent base_link, child rear_right_wheel, origin xyz=-0.25 -0.28 0 rpy=0 0 0, axis 0 1 0
